Commit message: added lidar

File: src/agv_description/urdf/agv.urdf (robot description, URDF)
Before this commit: robot warehouse_agv, 5 links, 4 joints
Links:
- removed link caster_wheel
- added link camera_optical_frame
- added link front_caster, mass 0.08; collision sphere radius=0.025; visual sphere radius=0.025
- added link lidar_link, mass 0.18; collision cylinder length=0.06 radius=0.04; visual cylinder length=0.06 radius=0.04
- added link rear_caster, mass 0.08; collision sphere radius=0.025; visual sphere radius=0.025
- added link top_deck, mass 0.1; visual cylinder length=0.008 radius=0.21
- link base_link: mass 5.0 -> 8.0; geometry collision cylinder length=0.12 radius=0.22; visual cylinder length=0.12 radius=0.22
- link camera_link: mass None -> 0.05; geometry collision box size=0.02 0.06 0.025; visual box size=0.02 0.06 0.025
- link left_wheel: mass 0.5 -> 0.4; geometry collision cylinder length=0.04 radius=0.05; visual cylinder length=0.04 radius=0.05
- link right_wheel: mass 0.5 -> 0.4; geometry collision cylinder length=0.04 radius=0.05; visual cylinder length=0.04 radius=0.05
Joints:
- removed joint caster_wheel_joint
- added joint camera_optical_joint: type fixed, parent camera_link, child camera_optical_frame, origin xyz=0 0 0 rpy=-1.5708 0 -1.5708
- added joint front_caster_joint: type fixed, parent base_link, child front_caster, origin xyz=0.17 0.0 -0.06 rpy=0 0 0
- added joint lidar_joint: type fixed, parent base_link, child lidar_link, origin xyz=0.0 0.0 0.09 rpy=0 0 0
- added joint rear_caster_joint: type fixed, parent base_link, child rear_caster, origin xyz=-0.17 0.0 -0.06 rpy=0 0 0
- added joint top_deck_joint: type fixed, parent base_link, child top_deck, origin xyz=0.0 0.0 0.064 rpy=0 0 0
- joint camera_joint: origin xyz=0.3 0 0.1 rpy=0 0 0 -> xyz=0.21 0.0 0.01 rpy=0 0 0
- joint left_wheel_joint: origin xyz=0.15 0.225 -0.05 rpy=-1.5708 0 0 -> xyz=0.0 0.245 -0.035 rpy=-1.5708 0 0
- joint right_wheel_joint: origin xyz=0.15 -0.225 -0.05 rpy=1.5708 0 0 -> xyz=0.0 -0.245 -0.035 rpy=1.5708 0 0

Commit message: Revert "added lidar"
This reverts commit 10feb98107110bcf20bada76bbf48cd2f01d7876.

File: src/agv_description/urdf/agv.urdf (robot description, URDF)
Before this commit: robot warehouse_agv, 9 links, 8 joints
Links:
- removed link camera_optical_frame
- removed link front_caster
- removed link lidar_link
- removed link rear_caster
- removed link top_deck
- added link caster_wheel, mass 0.1; collision sphere radius=0.05; visual sphere radius=0.05
- link base_link: mass 8.0 -> 5.0; geometry collision box size=0.6 0.4 0.2; visual box size=0.6 0.4 0.2
- link camera_link: mass 0.05 -> None; geometry visual box size=0.02 0.05 0.05
- link left_wheel: mass 0.4 -> 0.5; geometry collision cylinder length=0.05 radius=0.1; visual cylinder length=0.05 radius=0.1
- link right_wheel: mass 0.4 -> 0.5; geometry collision cylinder length=0.05 radius=0.1; visual cylinder length=0.05 radius=0.1
Joints:
- removed joint camera_optical_joint
- removed joint front_caster_joint
- removed joint lidar_joint
- removed joint rear_caster_joint
- removed joint top_deck_joint
- added joint caster_wheel_joint: type fixed, parent base_link, child caster_wheel, origin xyz=-0.2 0 -0.1 rpy=0 0 0
- joint camera_joint: origin xyz=0.21 0.0 0.01 rpy=0 0 0 -> xyz=0.3 0 0.1 rpy=0 0 0
- joint left_wheel_joint: origin xyz=0.0 0.245 -0.035 rpy=-1.5708 0 0 -> xyz=0.15 0.225 -0.05 rpy=-1.5708 0 0
- joint right_wheel_joint: origin xyz=0.0 -0.245 -0.035 rpy=1.5708 0 0 -> xyz=0.15 -0.225 -0.05 rpy=1.5708 0 0
