Commit message: moving for some distance and crashing

File: src/agv_description/urdf/warehouse_agv.urdf (robot description, URDF)
Before this commit: robot warehouse_agv, 8 links, 7 joints
Links:
- link base_link: geometry collision cylinder length=0.12 radius=0.15; visual cylinder length=0.12 radius=0.15
Joints:
- joint left_wheel_joint: origin xyz=0 0.23 0.05 -> xyz=0 0.17 0.05
- joint right_wheel_joint: origin xyz=0 -0.23 0.05 -> xyz=0 -0.17 0.05

Commit message: Revert "moving for some distance and crashing"
This reverts commit 710bccebc73c48cee6b366f10a555d95327ac9e4.

File: src/agv_description/urdf/warehouse_agv.urdf (robot description, URDF)
Before this commit: robot warehouse_agv, 8 links, 7 joints
Links:
- link base_link: geometry collision cylinder length=0.12 radius=0.22; visual cylinder length=0.12 radius=0.22
Joints:
- joint left_wheel_joint: origin xyz=0 0.17 0.05 -> xyz=0 0.23 0.05
- joint right_wheel_joint: origin xyz=0 -0.17 0.05 -> xyz=0 -0.23 0.05

Commit message: running success

File: src/agv_description/urdf/warehouse_agv.urdf (robot description, URDF)
Before this commit: robot warehouse_agv, 8 links, 7 joints
Links:
- link base_link: geometry collision cylinder length=0.12 radius=0.15; visual cylinder length=0.12 radius=0.15
Joints:
- joint camera_joint: origin xyz=0.22 0 0.06 -> xyz=0.15 0 0.06
- joint front_caster_joint: origin xyz=0.18 0 0.025 -> xyz=0.12 0 0.025
- joint left_wheel_joint: axis 0 -1 0 -> 0 1 0; origin xyz=0 0.23 0.05 -> xyz=0 0.17 0.05
- joint rear_caster_joint: origin xyz=-0.18 0 0.025 -> xyz=-0.12 0 0.025
- joint right_wheel_joint: axis 0 -1 0 -> 0 1 0; origin xyz=0 -0.23 0.05 -> xyz=0 -0.17 0.05

Commit message: mapping done, only fine tuning required more precision

File: src/agv_description/urdf/warehouse_agv.urdf (robot description, URDF)
Before this commit: robot warehouse_agv, 8 links, 7 joints
Joints:
- joint camera_joint: origin xyz=0.15 0 0.06 -> xyz=0.15 0 0.07
- joint imu_joint: origin xyz=0 0 0.06 -> xyz=0 0 0.07
- joint lidar_joint: origin xyz=0 0 0.145 -> xyz=0 0 0.155
