Commit message: changes made to dimension and works well

File: src/agv_description/urdf/warehouse_agv.urdf (robot description, URDF)
Before this commit: robot warehouse_agv, 7 links, 6 joints
Links:
- link base_link: mass 12.0 -> 8.0; geometry collision cylinder length=0.10 radius=0.11; visual cylinder length=0.10 radius=0.11
- link front_caster: mass 0.5 -> 0.2
- link left_wheel: mass 2.0 -> 1.0; geometry collision cylinder length=0.03 radius=0.025; visual cylinder length=0.03 radius=0.025
- link rear_caster: mass 0.5 -> 0.2
- link right_wheel: mass 2.0 -> 1.0; geometry collision cylinder length=0.03 radius=0.025; visual cylinder length=0.03 radius=0.025
Joints:
- joint front_caster_joint: origin xyz=0.12 0 0.025 -> xyz=0.09 0 0.025
- joint imu_joint: origin xyz=0 0 0.07 -> xyz=0 0 0.06
- joint left_wheel_joint: origin xyz=0 0.17 0.05 -> xyz=0 0.13 0.025
- joint lidar_joint: origin xyz=0 0 0.155 -> xyz=0 0 0.135
- joint rear_caster_joint: origin xyz=-0.12 0 0.025 -> xyz=-0.09 0 0.025
- joint right_wheel_joint: origin xyz=0 -0.17 0.05 -> xyz=0 -0.13 0.025
