Commit message: odometry added

File: install/agv_description/share/agv_description/urdf/warehouse_agv.urdf (robot description, URDF)
Before this commit: robot warehouse_agv, 6 links, 5 joints
Links:
- added link imu_link, mass 0.1
Joints:
- added joint imu_joint: type fixed, parent base_link, child imu_link, origin xyz=0 0 0.05

File: src/agv_description/urdf/warehouse_agv.urdf (robot description, URDF)
Before this commit: robot warehouse_agv, 6 links, 5 joints
Links:
- added link imu_link, mass 0.1
Joints:
- added joint imu_joint: type fixed, parent base_link, child imu_link, origin xyz=0 0 0.05

Commit message: added camera

File: install/agv_description/share/agv_description/urdf/warehouse_agv.urdf (robot description, URDF)
Before this commit: robot warehouse_agv, 7 links, 6 joints
Links:
- added link camera_link, mass 0.1; collision box size=0.02 0.05 0.05; visual box size=0.02 0.05 0.05
Joints:
- added joint camera_joint: type fixed, parent base_link, child camera_link, origin xyz=0.26 0 0.10

Commit message: mapping with new robot model

File: install/agv_description/share/agv_description/urdf/warehouse_agv.urdf (robot description, URDF)
Before this commit: robot warehouse_agv, 8 links, 7 joints
Links:
- link base_link: geometry collision cylinder length=0.12 radius=0.22; visual cylinder length=0.12 radius=0.22
- link front_caster: geometry collision sphere radius=0.025; visual sphere radius=0.025
- link rear_caster: geometry collision sphere radius=0.025; visual sphere radius=0.025
Joints:
- joint camera_joint: origin xyz=0.26 0 0.10 -> xyz=0.22 0 0.06
- joint front_caster_joint: origin xyz=0.18 0 0.03 -> xyz=0.18 0 0.025
- joint imu_joint: origin xyz=0 0 0.05 -> xyz=0 0 0.06
- joint lidar_joint: origin xyz=0 0 0.13 -> xyz=0 0 0.145
- joint rear_caster_joint: origin xyz=-0.18 0 0.03 -> xyz=-0.18 0 0.025
